Commit message: Fix TF conflicts: remove Gazebo TF bridge, clean URDF frames, and stabilize transform tree, made the left arm fixed temporarily for compnent3

File: ros_gz_example_description/urdf/robot.urdf (robot description, URDF)
Before this commit: robot diff_drive, 20 links, 19 joints
Links:
- removed link base_footprint
Joints:
- removed joint base_footprint_joint
- joint elbow_joint: type revolute -> fixed
- joint shoulder_joint: type revolute -> fixed
- joint wrist_joint: type revolute -> fixed
